File: thermidity-kicad/thermidity.kicad_pcb (KiCad board)
At the start: 2 copper layers, 60 x 30 mm, 23 parts, among them J1 Battery, J2 Display, J3 ISP, U1 MCP1501-30, U2 ATmega328P, U3 TMP36, U4 HIH-5030

Commit message: ratiometric measurement of humidity
- update PCB
- measure battery voltage using internal 1.1V reference
Parts:
- removed C1, C4: 2.2uF, Capacitor_SMD:C_1206_3216Metric_Pad1.33x1.80mm_HandSolder
- removed R1: 68, Resistor_SMD:R_0805_2012Metric_Pad1.20x1.40mm_HandSolder
- removed R2: 51, Resistor_SMD:R_0805_2012Metric_Pad1.20x1.40mm_HandSolder
- removed the U1 at (125.5, 79.1)
- moved R4 2.54 mm to (137.7, 78.4), turned to 90 degrees
- moved R3 2.44 mm to (135.2, 78.4), turned to -90 degrees
- moved C5 0.81 mm to (135.2, 84.8), turned to 180 degrees
- moved R5 0.31 mm to (148.6, 84.9)
- turned U3 to 0 degrees
- renumbered R4 to R3, R3 to R4, U2 to U1, U4 to U2
Connections:
- C3 pad 2: Net-(C3-Pad2) -> Net-(U1-Pad20)
- C5 pad 1: +BATT -> Net-(C5-Pad1)
- R3 pad 1: Net-(U2-Pad24) -> Net-(U1-Pad23)
- R4 pad 1: +BATT -> Net-(C5-Pad1)
- R4 pad 2: Net-(U2-Pad24) -> Net-(U1-Pad23)
- U1 pad 20: Net-(C3-Pad2) -> Net-(U1-Pad20)
- U1 pad 23: Net-(U2-Pad23) -> Net-(U1-Pad23)
- U1 pad 24: Net-(U2-Pad24) -> Net-(C5-Pad1)
- U2 pad 3: Net-(C3-Pad2) -> Net-(C5-Pad1)
- U3 pad 1: +BATT -> Net-(C5-Pad1)
Routing:
- net Net-(C3-Pad2): track 49.8 -> 0.00 mm
- net +BATT: track 85.2 -> 47.2 mm, vias 4 -> 2
- net Net-(C5-Pad1): track 0.00 -> 28.5 mm
- net Net-(U2-Pad23): track 26.8 -> 0.00 mm, vias 2 -> 0
- net Net-(U2-Pad24): track 7.11 -> 0.00 mm
- net Net-(U1-Pad23): track 0.00 -> 6.61 mm
- net GND: track 24.6 -> 20.7 mm, vias 13 -> 8
- net Net-(C4-Pad1): track 3.94 -> 0.00 mm
- net Net-(U1-Pad20): track 0.00 -> 3.27 mm
- net Net-(C1-Pad2): track 3.23 -> 0.00 mm
- removed copper zone on F.Cu, net GND
