File: thermidity-kicad/thermidity.kicad_pcb (KiCad board)
At the start: 2 copper layers, 60 x 30 mm, 18 parts, among them J1 Battery, J2 Display, J3 ISP, U1 ATmega328P, U2 HIH-5030

Commit message: disable SPI between display updates, fix schematic
- fix high power consumption of display in sleep mode by disabling SPI (driving SCK low)
- remove "unconnected" from MCU pin 20 (AREF) as it is connected
- update README and manual
Connections:
- C2 pad 2: unconnected-(U1-Pad20) -> Net-(C2-Pad2)
- U1 pad 20: unconnected-(U1-Pad20) -> Net-(C2-Pad2)
Routing:
- net unconnected-(U1-Pad20): track 3.28 -> 0.00 mm
- net Net-(C2-Pad2): track 0.00 -> 3.28 mm
Changed lines of the file:
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@@
   (net 14 "Net-(J3-Pad2)")
   (net 15 "Net-(R2-Pad1)")
-  (net 16 "unconnected-(U1-Pad20)")
+  (net 16 "Net-(C2-Pad2)")
   (net 17 "unconnected-(U1-Pad1)")
   (net 18 "unconnected-(U1-Pad2)")
@@
   (net 22 "unconnected-(U1-Pad19)")
   (net 23 "unconnected-(U1-Pad22)")
-  (net 24 "Net-(U1-Pad25)")
+  (net 24 "Net-(R3-Pad1)")
   (net 25 "unconnected-(U1-Pad27)")
   (net 26 "unconnected-(U1-Pad28)")
@@
       (net 15 "Net-(R2-Pad1)") (pintype "passive"))
     (pad "2" smd roundrect (at 1 0) (size 1.2 1.4) (layers "F.Cu" "F.Paste" "F.Mask") (roundrect_rratio 0.208333)
-      (net 24 "Net-(U1-Pad25)") (pintype "passive"))
+      (net 24 "Net-(R3-Pad1)") (pintype "passive"))
     (model "${KICAD6_3DMODEL_DIR}/Resistor_SMD.3dshapes/R_0805_2012Metric.wrl"
       (offset (xyz 0 0 0))
@@
       (net 22 "unconnected-(U1-Pad19)") (pinfunction "ADC6") (pintype "input+no_connect"))
     (pad "20" smd rect (at 4.25 0.4 180) (size 1.6 0.55) (layers "F.Cu" "F.Paste" "F.Mask")
-      (net 16 "unconnected-(U1-Pad20)") (pinfunction "AREF") (pintype "passive+no_connect"))
+      (net 16 "Net-(C2-Pad2)") (pinfunction "AREF") (pintype "passive"))
     (pad "21" smd rect (at 4.25 -0.4 180) (size 1.6 0.55) (layers "F.Cu" "F.Paste" "F.Mask")
       (net 1 "GND") (pinfunction "GND") (pintype "passive"))
@@
       (net 15 "Net-(R2-Pad1)") (pinfunction "PC1") (pintype "bidirectional"))
     (pad "25" smd rect (at 2.8 -4.25 270) (size 1.6 0.55) (layers "F.Cu" "F.Paste" "F.Mask")
-      (net 24 "Net-(U1-Pad25)") (pinfunction "PC2") (pintype "bidirectional"))
+      (net 24 "Net-(R3-Pad1)") (pinfunction "PC2") (pintype "bidirectional"))
     (pad "26" smd rect (at 2 -4.25 270) (size 1.6 0.55) (layers "F.Cu" "F.Paste" "F.Mask")
       (net 32 "Net-(R4-Pad1)") (pinfunction "PC3") (pintype "bidirectional"))
@@
     (fp_line (start -1 -0.625) (end 1 -0.625) (layer "F.Fab") (width 0.1))
     (pad "1" smd roundrect (at -1 0) (size 1.2 1.4) (layers "F.Cu" "F.Paste" "F.Mask") (roundrect_rratio 0.208333)
-      (net 24 "Net-(U1-Pad25)") (pintype "passive"))
+      (net 24 "Net-(R3-Pad1)") (pintype "passive"))
     (pad "2" smd roundrect (at 1 0) (size 1.2 1.4) (layers "F.Cu" "F.Paste" "F.Mask") (roundrect_rratio 0.208333)
       (net 1 "GND") (pintype "passive"))
@@
       (net 1 "GND") (pintype "passive"))
     (pad "2" smd roundrect (at 1.5625 0) (size 1.325 1.8) (layers "F.Cu" "F.Paste" "F.Mask") (roundrect_rratio 0.188679)
-      (net 16 "unconnected-(U1-Pad20)") (pintype "passive+no_connect"))
+      (net 16 "Net-(C2-Pad2)") (pintype "passive"))
     (model "${KICAD6_3DMODEL_DIR}/Capacitor_SMD.3dshapes/C_1206_3216Metric.wrl"
       (offset (xyz 0 0 0))
