File: thermidity-kicad/thermidity.kicad_sch (KiCad schematic)
At the start: 13 parts, among them J1 Battery, J2 Display, J3 ISP, U1 ATmega328P, U2 HIH-5030, U3 TMP36

Commit message: ratiometric measurement of temperature
- replace TMP36 with a thermistor NTC 100k
- put back 1nF cap between AREF and GND
- wait 150us for the cap to discharge before converting with 1.1V reference
- uint16_t is enough for 16x ADC
Parts:
- removed C3: 100nF, Capacitor_SMD:C_1206_3216Metric_Pad1.33x1.80mm_HandSolder, symbol Device:C
- removed U3: TMP36, TMP36GT9:XDCR_TMP36GT9, symbol TMP36GT9:TMP36GT9
- added C2: 1nF, Capacitor_SMD:C_1206_3216Metric_Pad1.33x1.80mm_HandSolder, symbol Device:C
- added R3: 100k, Resistor_SMD:R_0805_2012Metric_Pad1.20x1.40mm_HandSolder, symbol Device:R
- added TH1: NTC 100k, Resistor_THT:R_Axial_DIN0204_L3.6mm_D1.6mm_P2.54mm_Vertical, symbol Device:Thermistor_NTC
- R1: value 1M -> 300K
- R2: value 1M -> 1.2M
- renumbered C2 to C3, R3 to R4
Connections:
- net GND: now also C2.1, R3.2
- net at R2.1, U1.24 (PC1), U2.3 (+VE): now also TH1.1
- net at U1.20 (AREF): now also C2.2
- net at U1.25 (PC2): now also R3.1, TH1.2

Commit message: ratiometric measurement of temperature
- SMD footprint instead of TH for thermistor
Parts:
- TH1: footprint Resistor_THT:R_Axial_DIN0204_L3.6mm_D1.6mm_P2.54mm_Vertical -> Resistor_SMD:R_1206_3216Metric_Pad1.30x1.75mm_HandSolder
Changed lines of the file:
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@@
       (effects (font (size 1.27 1.27)) (justify left))
     )
-    (property "Footprint" "Resistor_THT:R_Axial_DIN0204_L3.6mm_D1.6mm_P2.54mm_Vertical" (id 2) (at 186.69 38.1 0)
+    (property "Footprint" "Resistor_SMD:R_1206_3216Metric_Pad1.30x1.75mm_HandSolder" (id 2) (at 186.69 38.1 0)
       (effects (font (size 1.27 1.27)) hide)
     )
@@
     )
     (path "/982b487a-58ee-40be-91ad-fe1876106c60"
-      (reference "TH1") (unit 1) (value "NTC 100k") (footprint "Resistor_THT:R_Axial_DIN0204_L3.6mm_D1.6mm_P2.54mm_Vertical")
+      (reference "TH1") (unit 1) (value "NTC 100k") (footprint "Resistor_SMD:R_1206_3216Metric_Pad1.30x1.75mm_HandSolder")
     )
     (path "/a564f624-0149-43d3-9b25-20abc178b1e7"

Commit message: ratiometric measurement of temperature
- calculate temperature
- rounding of temperature compensated relative humidity
- no need for battery voltage in mV
Parts:
- TH1: footprint Resistor_SMD:R_1206_3216Metric_Pad1.30x1.75mm_HandSolder -> Resistor_SMD:R_0805_2012Metric_Pad1.20x1.40mm_HandSolder
Changed lines of the file:
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@@
       (effects (font (size 1.27 1.27)) (justify left))
     )
-    (property "Footprint" "Resistor_SMD:R_1206_3216Metric_Pad1.30x1.75mm_HandSolder" (id 2) (at 186.69 38.1 0)
+    (property "Footprint" "Resistor_SMD:R_0805_2012Metric_Pad1.20x1.40mm_HandSolder" (id 2) (at 186.69 38.1 0)
       (effects (font (size 1.27 1.27)) hide)
     )
@@
     )
     (path "/982b487a-58ee-40be-91ad-fe1876106c60"
-      (reference "TH1") (unit 1) (value "NTC 100k") (footprint "Resistor_SMD:R_1206_3216Metric_Pad1.30x1.75mm_HandSolder")
+      (reference "TH1") (unit 1) (value "NTC 100k") (footprint "Resistor_SMD:R_0805_2012Metric_Pad1.20x1.40mm_HandSolder")
     )
     (path "/a564f624-0149-43d3-9b25-20abc178b1e7"
